File: User Interface.kicad_sch (KiCad schematic)
At the start: 4 parts, among them SW1 SW_DIP_x01, U1 7400, U2 7402

Commit message: 3 How To Design A Circuit Using KiCad 7.0 Schematic Editor
https://www.youtube.com/watch?v=pgKfaFI4T4Y
Parts:
- removed SW1: SW_DIP_x01, symbol Switch:SW_DIP_x01
- removed U1: 7400, symbol 74xx:7400
- removed U2: 7402, symbol 74xx:7402
- added BT1: Battery_Cell, symbol Device:Battery_Cell
- added MK1: Microphone_Condenser, symbol Device:Microphone_Condenser
- added R1, R2, R3: R, symbol Device:R
- added R4: LDR07, OptoDevice:R_LDR_5.1x4.3mm_P3.4mm_Vertical, symbol Sensor_Optical:LDR07
- added SW1: SW_DPDT_x2, symbol Switch:SW_DPDT_x2
- added U1: ATtiny85V-10P, Package_DIP:DIP-8_W7.62mm, symbol MCU_Microchip_ATtiny:ATtiny85V-10P
Connections:
- net GND: now also MK1.1 (-), R1.2, R4.2, SW1.2 (B), U1.4 (GND); no longer D1.1 (K)
- net at D1.2 (A): now also U1.6 (PB1)
- new net: D1.1 (K), R1.1
- new net: MK1.2 (+), R2.2, U1.7 (PB2)
- new net: R3.2, R4.1, U1.3 (XTAL2/PB4)
- new net: BT1.2 (-), SW1.3 (C)
- new net +3.3V: BT1.1 (+), R2.1, R3.1, U1.8 (VCC)

Commit message: 4 How To Prettify Your Schematic with Kicad 7.0
https://www.youtube.com/watch?v=iqIRjMkHVjY
Parts:
- BT1: value Battery_Cell -> 3.3V Cell
- D1: value LED -> 5mm Yellow LED
- R1: renamed from R3; value R -> 10k
- R2: renamed from R4; value LDR07 -> 5mm LDR
- R3: renamed from R2; value R -> 5.6k
- R4: renamed from R1; value R -> 470R
- SW1: value SW_DPDT_x2 -> Slide Switch
Connections:
- net LED: now reaches D1.2 (A), U1.6 (PB1)
- net MIC: now reaches MK1.2 (+), R3.2
- net MIC: now also U1.2 (XTAL1/PB3); no longer U1.7 (PB2)
- net LDR: now reaches R1.2, R2.1
- net LDR: now also U1.7 (PB2); no longer U1.3 (XTAL2/PB4)
- no-connect marks 0 -> 3
Other:
- note added: "Battery Unit"
- note added: "LDR Unit"
- note added: "Ligth Unit"
- note added: "Microcontroller Unit"
- note added: "Sound Sensing Unit"
- company: (none) -> It's a ATTiny 85 Based Circuit
- title: (none) -> Digital Diya
- moved on the sheet: BT1, D1, MK1, R1, R2, R3, R4, SW1A, U1

Commit message: 5 How To Perform ERC and What Is Footprint In KiCad 7.0
https://www.youtube.com/watch?v=A5uNG_jQ4qM
Parts:
- removed SW1: Slide Switch, symbol Switch:SW_DPDT_x2
- added SW1: SW_SPDT, symbol Switch:SW_SPDT
Connections:
- net GND: now also SW1.2 (B)
- net at BT1.2 (-): now also SW1.3 (C)
- no-connect marks 3 -> 4
Changed lines of the file:
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@@
+	)
+	(junction
+		(at 64.77 85.09)
+		(diameter 0)
+		(color 0 0 0 0)
+	)
+	(junction
+		(at 62.23 107.95)
+		(diameter 0)
+		(color 0 0 0 0)
 	)
 	(junction
@@
 	)
 	(no_connect
+		(at 59.69 96.52)
+	)
+	(no_connect
 		(at 129.54 105.41)
 	)
@@
 	(wire
 		(pts
-			(xy 62.23 106.68) (xy 62.23 109.22)
+			(xy 64.77 85.09) (xy 64.77 86.36)
+		)
+		(stroke
+			(width 0)
+			(type default)
+		)
+	)
+	(wire
+		(pts
+			(xy 62.23 106.68) (xy 62.23 107.95)
 		)
 		(stroke
@@
 	(wire
 		(pts
-			(xy 64.77 83.82) (xy 64.77 86.36)
+			(xy 64.77 85.09) (xy 73.66 85.09)
+		)
+		(stroke
+			(width 0)
+			(type default)
+		)
+	)
+	(wire
+		(pts
+			(xy 64.77 83.82) (xy 64.77 85.09)
 		)
 		(stroke
@@
 	(wire
 		(pts
+			(xy 62.23 107.95) (xy 62.23 109.22)
+		)
+		(stroke
+			(width 0)
+			(type default)
+		)
+	)
+	(wire
+		(pts
 			(xy 182.88 95.25) (xy 191.77 95.25)
 		)
@@
 		(pts
 			(xy 114.3 115.57) (xy 114.3 118.11)
+		)
+		(stroke
+			(width 0)
+			(type default)
+		)
+	)
+	(wire
+		(pts
+			(xy 62.23 107.95) (xy 73.66 107.95)
 		)
 		(stroke
@@
 	)
 	(symbol
+		(lib_id "Switch:SW_SPDT")
+		(at 62.23 101.6 90)
+		(unit 1)
+		(exclude_from_sim no)
+		(in_bom yes)
+		(on_board yes)
+		(dnp no)
+		(fields_autoplaced yes)
+		(property "Reference" "SW1"
+			(at 67.31 100.3299 90)
+			(effects
+				(font
+					(size 1.27 1.27)
+				)
+				(justify right)
+			)
+		)
+		(property "Value" "SW_SPDT"
+			(at 67.31 102.8699 90)
+			(effects
+				(font
+					(size 1.27 1.27)
+				)
+				(justify right)
+			)
+		)
+		(property "Footprint" ""
+			(at 62.23 101.6 0)
+			(effects
+				(font
+					(size 1.27 1.27)
+				)
+				(hide yes)
+			)
+		)
+		(property "Datasheet" "~"
+			(at 69.85 101.6 0)
+			(effects
+				(font
+					(size 1.27 1.27)
+				)
+				(hide yes)
+			)
+		)
+		(property "Description" "Switch, single pole double throw"
+			(at 62.23 101.6 0)
+			(effects
+				(font
+					(size 1.27 1.27)
+				)
+				(hide yes)
+			)
+		)
+		(pin "2"
+		)
+		(pin "1"
+		)
+		(pin "3"
+		)
+		(instances
+			(project "User Interface"
+				(path "/b2c2918b-4aac-4a65-b902-923319962657"
+					(reference "SW1")
+					(unit 1)
+				)
+			)
+		)
+	)
+	(symbol
 		(lib_id "Device:LED")
 		(at 227.33 92.71 90)
@@
 	)
 	(symbol
+		(lib_id "power:PWR_FLAG")
+		(at 73.66 107.95 180)
+		(unit 1)
+		(exclude_from_sim no)
+		(in_bom yes)
+		(on_board yes)
+		(dnp no)
+		(fields_autoplaced yes)
+		(property "Reference" "#FLG02"
+			(at 73.66 109.855 0)
+			(effects
+				(font
+					(size 1.27 1.27)
+				)
+				(hide yes)
+			)
+		)
+		(property "Value" "PWR_FLAG"
+			(at 73.66 113.03 0)
+			(effects
+				(font
+					(size 1.27 1.27)
+				)
+			)
+		)
+		(property "Footprint" ""
+			(at 73.66 107.95 0)
+			(effects
+				(font
+					(size 1.27 1.27)
+				)
+				(hide yes)
+			)
+		)
+		(property "Datasheet" "~"
+			(at 73.66 107.95 0)
+			(effects
+				(font
+					(size 1.27 1.27)
+				)
+				(hide yes)
+			)
+		)
+		(property "Description" "Special symbol for telling ERC where power comes from"
+			(at 73.66 107.95 0)
+			(effects
+				(font
+					(size 1.27 1.27)
+				)
+				(hide yes)
+			)
+		)
+		(pin "1"
+		)
+		(instances
+			(project "User Interface"
+				(path "/b2c2918b-4aac-4a65-b902-923319962657"
+					(reference "#FLG02")
+					(unit 1)
+				)
+			)
+		)
+	)
+	(symbol
 		(lib_id "Device:Microphone_Condenser")
 		(at 191.77 102.87 0)
@@
 	)
 	(symbol
-		(lib_id "Switch:SW_DPDT_x2")
-		(at 62.23 101.6 90)
-		(unit 1)
-		(exclude_from_sim no)
-		(in_bom yes)
-		(on_board yes)
-		(dnp no)
-		(fields_autoplaced yes)
-		(property "Reference" "SW1"
-			(at 67.31 100.3299 90)
-			(effects
-				(font
-					(size 1.27 1.27)
-				)
-				(justify right)
-			)
-		)
-		(property "Value" "Slide Switch"
-			(at 67.31 102.8699 90)
-			(effects
-				(font
-					(size 1.27 1.27)
-				)
-				(justify right)
-			)
-		)
-		(property "Footprint" ""
-			(at 62.23 101.6 0)
-			(effects
-				(font
-					(size 1.27 1.27)
-				)
-				(hide yes)
-			)
-		)
-		(property "Datasheet" "~"
-			(at 62.23 101.6 0)
-			(effects
-				(font
-					(size 1.27 1.27)
-				)
-				(hide yes)
-			)
-		)
-		(property "Description" "Switch, dual pole double throw, separate symbols"
-			(at 62.23 101.6 0)
-			(effects
-				(font
-					(size 1.27 1.27)
-				)
-				(hide yes)
-			)
-		)
-		(pin "1"
-		)
-		(pin "2"
-		)
-		(pin "3"
-		)
-		(pin "5"
-		)
-		(pin "6"
-		)
-		(pin "4"
-		)
-		(instances
-			(project "User Interface"
-				(path "/b2c2918b-4aac-4a65-b902-923319962657"
-					(reference "SW1")
-					(unit 1)
-				)
-			)
-		)
-	)
-	(symbol
 		(lib_id "Device:Battery_Cell")
 		(at 64.77 91.44 0)
@@
 					(unit 1)
 				)
+			)
+		)
+	)
+	(symbol
+		(lib_id "power:PWR_FLAG")
+		(at 73.66 85.09 0)
+		(unit 1)
+		(exclude_from_sim no)
+		(in_bom yes)
+		(on_board yes)
+		(dnp no)
+		(fields_autoplaced yes)
+		(property "Reference" "#FLG01"
+			(at 73.66 83.185 0)
+			(effects
+				(font
+					(size 1.27 1.27)
+				)
+				(hide yes)
+			)
+		)
+		(property "Value" "PWR_FLAG"
+			(at 73.66 80.01 0)
+			(effects
+				(font
+					(size 1.27 1.27)
+				)
+			)
+		)
+		(property "Footprint" ""
+			(at 73.66 85.09 0)
+			(effects
+				(font
+					(size 1.27 1.27)
+				)
+				(hide yes)
+			)
+		)
+		(property "Datasheet" "~"
+			(at 73.66 85.09 0)
+			(effects
+				(font
+					(size 1.27 1.27)
+				)
+				(hide yes)
+			)
+		)
+		(property "Description" "Special symbol for telling ERC where power comes from"
+			(at 73.66 85.09 0)
+			(effects
+				(font
+					(size 1.27 1.27)
+				)
+				(hide yes)
+			)
+		)
+		(pin "1"
+		)
+		(instances
+			(project "User Interface"
+				(path "/b2c2918b-4aac-4a65-b902-923319962657"
+					(reference "#FLG01")
+					(unit 1)
+				)

Commit message: 6 How To Select The Right Footprint For Symbols in KiCad 7.0
https://www.youtube.com/watch?v=JMa9q4YhRDk
Parts:
- BT1: footprint (none) -> Battery:BatteryHolder_ComfortableElectronic_CH273-2450_1x2450
- D1: footprint (none) -> LED_THT:LED_D5.0mm
- MK1: footprint (none) -> Connector_PinHeader_2.54mm:PinHeader_1x02_P2.54mm_Vertical
- R1, R3, R4: footprint (none) -> Resistor_THT:R_Axial_DIN0207_L6.3mm_D2.5mm_P15.24mm_Horizontal
- SW1: footprint (none) -> Button_Switch_THT:SW_E-Switch_EG1224_SPDT_Angled
Changed lines of the file:
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@@
 			)
 		)
-		(property "Footprint" ""
+		(property "Footprint" "Button_Switch_THT:SW_E-Switch_EG1224_SPDT_Angled"
 			(at 62.23 101.6 0)
 			(effects
@@
 			)
 		)
-		(property "Footprint" ""
+		(property "Footprint" "LED_THT:LED_D5.0mm"
 			(at 227.33 92.71 0)
 			(effects
@@
 			)
 		)
-		(property "Footprint" ""
+		(property "Footprint" "Connector_PinHeader_2.54mm:PinHeader_1x02_P2.54mm_Vertical"
 			(at 191.77 100.33 90)
 			(effects
@@
 			)
 		)
-		(property "Footprint" ""
+		(property "Footprint" "Resistor_THT:R_Axial_DIN0207_L6.3mm_D2.5mm_P15.24mm_Horizontal"
 			(at 189.992 88.9 90)
 			(effects
@@
 			)
 		)
-		(property "Footprint" ""
+		(property "Footprint" "Battery:BatteryHolder_ComfortableElectronic_CH273-2450_1x2450"
 			(at 64.77 89.916 90)
 			(effects
@@
 			)
 		)
-		(property "Footprint" ""
+		(property "Footprint" "Resistor_THT:R_Axial_DIN0207_L6.3mm_D2.5mm_P15.24mm_Horizontal"
 			(at 225.552 102.87 90)
 			(effects
@@
 			)
 		)
-		(property "Footprint" ""
+		(property "Footprint" "Resistor_THT:R_Axial_DIN0207_L6.3mm_D2.5mm_P15.24mm_Horizontal"
 			(at 150.622 92.71 90)
 			(effects
